File: v02 - artigo/Ref_fixa_v02.kicad_pcb (KiCad board)
At the start: 2 copper layers, 84 x 69.5 mm, 69 parts, among them U1 LM358, U2 LM317AT, U3 LM337T, U4 REF102BP, U5 INA2133UA, U6 INA2133UA

Commit message: Changes in values
Change in R7 value, from 330 to 100. Change the voltage from -2.13 to
-1.52
Parts:
- R7: value 330 -> 100
Changed lines of the file:
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@@
       (effects (font (size 1 1) (thickness 0.15)))
     )
-    (fp_text value 330 (at 0 0 90) (layer F.Fab)
+    (fp_text value 100 (at 0 0 90) (layer F.Fab)
       (effects (font (size 1 1) (thickness 0.15)))
     )
